File: bindec/bindec.kicad_sch (KiCad schematic)
At the start: 35 parts, among them J1 Conn_02x05_Top_Bottom, J2 C1, J3 C2, J4 CLOCK, J5 C3, J6 C4, J7 Carry, SW1 SW_SPDT, SW2 SW_SPDT, SW3 SW_SPDT, U1 L7805, U2 4029, U3 ICM7555

Commit message: update
Parts:
- C1, C2, C5: footprint Capacitor_THT:C_Disc_D4.7mm_W2.5mm_P5.00mm -> benjiaomodular:Capacitor_Disc_D3.8mm_W2.6mm_P2.50mm
- C3, C4: footprint Capacitor_THT:CP_Radial_D6.3mm_P2.50mm -> benjiaomodular:Capacitor_Radial_D5.0mm_P2.5mm
- J1: footprint Connector_PinHeader_1.00mm:PinHeader_2x05_P1.00mm_Vertical -> Connector_IDC:IDC-Header_2x05_P2.54mm_Vertical; symbol Connector_Generic:Conn_02x05_Top_Bottom -> Connector_Generic:Conn_02x05_Odd_Even
- J2, J3, J4, J5, J6, J7: footprint Connector_Audio:Jack_3.5mm_QingPu_WQP-PJ398SM_Vertical_CircularHoles -> benjiaomodular:AudioJack_3.5mm
- R1, R2, R3, R4, R5, R6, R7, R8, R9: footprint Resistor_THT:R_Axial_DIN0207_L6.3mm_D2.5mm_P10.16mm_Horizontal -> benjiaomodular:Resistor_L6.3mm_D2.5mm_P7.62mm_Horizontal
- RV1: footprint Potentiometer_THT:Potentiometer_Alpha_RD901F-40-00D_Single_Vertical -> benjiaomodular:Potentiometer_RV09
- SW1, SW2, SW3: footprint Connector_PinHeader_1.00mm:PinHeader_1x03_P1.00mm_Vertical -> Connector_PinSocket_2.54mm:PinSocket_1x03_P2.54mm_Vertical
Connections:
- net GND: now also J1.5 (Pin_5), J1.6 (Pin_6); no longer J1.2 (Pin_2), J1.9 (Pin_9)
- net at D1.2 (A), J1.1 (Pin_1): now also J1.2 (Pin_2); no longer J1.6 (Pin_6)
