File: bindec/bindec.kicad_pcb (KiCad board)
At the start: 2 copper layers, 40.3 x 128.5 mm, 4 parts

Commit message: update
Parts:
- added C1: 22u, benjiaomodular:Capacitor_Disc_D3.8mm_W2.6mm_P2.50mm, F.Cu at (229.0, 67.6)
- added C2: 100n, benjiaomodular:Capacitor_Disc_D3.8mm_W2.6mm_P2.50mm, F.Cu at (239.0, 62.1)
- added C3: 10u, benjiaomodular:Capacitor_Radial_D5.0mm_P2.5mm, F.Cu at (222.9, 68.5)
- added C4: 1u, benjiaomodular:Capacitor_Radial_D5.0mm_P2.5mm, F.Cu at (233.7, 56.7)
- added C5: 100n, benjiaomodular:Capacitor_Disc_D3.8mm_W2.6mm_P2.50mm, F.Cu at (210.8, 90.4)
- added D1: BAT85, Diode_THT:D_DO-35_SOD27_P7.62mm_Horizontal, F.Cu at (173.5, 91.4)
- added D2: C1_LED, LED_THT:LED_D3.0mm, F.Cu at (134.6, 84.4)
- added D3: C2_LED, LED_THT:LED_D3.0mm, F.Cu at (148.6, 84.4)
- added D4: CL_LED, LED_THT:LED_D3.0mm, F.Cu at (120.1, 84.4)
- added D5: C3_LED, LED_THT:LED_D3.0mm, F.Cu at (120.1, 107.3)
- added D6: C4_LED, LED_THT:LED_D3.0mm, F.Cu at (134.6, 107.3)
- added D7: CARRY_LED, LED_THT:LED_D3.0mm, F.Cu at (148.6, 107.3)
- added J1: Conn_02x05_Top_Bottom, Connector_IDC:IDC-Header_2x05_P2.54mm_Vertical, F.Cu at (119.6, 30.7)
- added J2: C1, benjiaomodular:AudioJack_3.5mm, F.Cu at (135.9, 89.7)
- added J3: C2, benjiaomodular:AudioJack_3.5mm, F.Cu at (149.9, 89.7)
- added J4: CLOCK, benjiaomodular:AudioJack_3.5mm, F.Cu at (121.4, 89.7)
- added J5: C3, benjiaomodular:AudioJack_3.5mm, F.Cu at (121.4, 112.5)
- added J6: C4, benjiaomodular:AudioJack_3.5mm, F.Cu at (135.9, 112.5)
- added J7: Carry, benjiaomodular:AudioJack_3.5mm, F.Cu at (149.9, 112.5)
- added R1: 1k, benjiaomodular:Resistor_L6.3mm_D2.5mm_P7.62mm_Horizontal, F.Cu at (206.9, 80.8)
- added R2: 1k, benjiaomodular:Resistor_L6.3mm_D2.5mm_P7.62mm_Horizontal, F.Cu at (195.4, 84.2)
- added R3: 1k, benjiaomodular:Resistor_L6.3mm_D2.5mm_P7.62mm_Horizontal, F.Cu at (222.4, 59.1)
- added R4: 1k, benjiaomodular:Resistor_L6.3mm_D2.5mm_P7.62mm_Horizontal, F.Cu at (207.6, 76.7)
- added R5: 1k, benjiaomodular:Resistor_L6.3mm_D2.5mm_P7.62mm_Horizontal, F.Cu at (195.4, 88.3)
- added R6: 10k, benjiaomodular:Resistor_L6.3mm_D2.5mm_P7.62mm_Horizontal, F.Cu at (222.4, 63.2)
- added R7: 10k, benjiaomodular:Resistor_L6.3mm_D2.5mm_P7.62mm_Horizontal, F.Cu at (229.5, 47.4)
- added R8: 1k, benjiaomodular:Resistor_L6.3mm_D2.5mm_P7.62mm_Horizontal, F.Cu at (229.5, 51.4)
- added R9: 1k, benjiaomodular:Resistor_L6.3mm_D2.5mm_P7.62mm_Horizontal, F.Cu at (240.2, 47.4)
- added RV1: 250k, benjiaomodular:Potentiometer_RV09, F.Cu at (133.4, 47.1)
- added SW1: SW_SPDT, Connector_PinSocket_2.54mm:PinSocket_1x03_P2.54mm_Vertical, F.Cu at (149.9, 68.1)
- added SW2: SW_SPDT, Connector_PinSocket_2.54mm:PinSocket_1x03_P2.54mm_Vertical, F.Cu at (121.4, 68.1)
- added SW3: SW_SPDT, Connector_PinSocket_2.54mm:PinSocket_1x03_P2.54mm_Vertical, F.Cu at (135.9, 68.1)
- added U1: L7805, Package_TO_SOT_THT:TO-220-3_Vertical, F.Cu at (147.3, 47.2)
- added U2: 4029, Package_DIP:DIP-16_W7.62mm, F.Cu at (118.9, 60.2)
- added U3: ICM7555, Package_DIP:DIP-8_W7.62mm, F.Cu at (144.3, 60.4)
- moved ? 35.5 mm to (26.9, 155.2)
- moved ? 35.5 mm to (52.3, 32.7)
- moved ? 35.5 mm to (26.9, 32.7)
- moved ? 35.5 mm to (52.3, 155.2)
Other:
- board size 40.3 x 128.5 mm -> 136.5 x 133.6 mm

Commit message: 123
Parts:
- removed ? (x4): , 
- added REF**: PanelHole_ToggleSwitch_MTS-101, benjiaomodular:PanelHole_ToggleSwitch_MTS-101, F.Cu at (89.8, 77.5)
- added REF**: PanelHole_AudioJack_3.5mm, benjiaomodular:PanelHole_AudioJack_3.5mm, F.Cu at (89.8, 119.4)
- added REF**: PanelHole_AudioJack_3.5mm, benjiaomodular:PanelHole_AudioJack_3.5mm, F.Cu at (103.7, 96.5)
- added REF**: PanelHole_Potentiometer_RV09, benjiaomodular:PanelHole_Potentiometer_RV09, F.Cu at (87.3, 54.0)
- added REF**: PanelHole_AudioJack_3.5mm, benjiaomodular:PanelHole_AudioJack_3.5mm, F.Cu at (75.3, 96.5)
- added REF**: PanelHole_ToggleSwitch_MTS-101, benjiaomodular:PanelHole_ToggleSwitch_MTS-101, F.Cu at (103.7, 77.5)
- added REF**: PanelHole_ToggleSwitch_MTS-101, benjiaomodular:PanelHole_ToggleSwitch_MTS-101, F.Cu at (75.3, 77.3)
- added REF**: PanelHole_AudioJack_3.5mm, benjiaomodular:PanelHole_AudioJack_3.5mm, F.Cu at (103.7, 119.4)
- added REF**: PanelHole_AudioJack_3.5mm, benjiaomodular:PanelHole_AudioJack_3.5mm, F.Cu at (89.8, 96.5)
- added REF**: e, benjiaomodular:PanelHole_AudioJack_3.5mm, F.Cu at (75.3, 119.4)
- added REF**: Panel_8HP, benjiaomodular:Panel_8HP, F.Cu at (68.7, 18.0)
- moved R9 103.6 mm to (162.3, 115.6), turned to 90 degrees
- moved R8 103.5 mm to (148.2, 115.4), turned to 90 degrees
- moved C4 92.4 mm to (144.1, 79.4)
- moved R3 86.1 mm to (144.6, 96.3), turned to -90 degrees
- moved C2 83.0 mm to (157.3, 76.8), turned to 90 degrees
- moved C1 80.6 mm to (157.0, 31.5), turned to -90 degrees
- moved C3 78.9 mm to (144.1, 71.1)
- moved R4 75.0 mm to (134.0, 91.1), turned to 90 degrees
- moved R7 67.9 mm to (161.5, 48.5)
- moved R5 67.4 mm to (133.8, 115.8), turned to 90 degrees
- moved C5 64.0 mm to (167.1, 43.6)
- moved D1 62.9 mm to (152.1, 32.3), turned to 180 degrees
- moved R6 61.8 mm to (161.5, 52.3)
- moved R1 59.3 mm to (148.4, 90.8), turned to 90 degrees
- moved R2 33.8 mm to (162.3, 91.1), turned to 90 degrees
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Routing:
- net GND: track 0.00 -> 256.2 mm
- net +5V: track 0.00 -> 83.1 mm
- net Q3: track 0.00 -> 77.2 mm
- net CARRY: track 0.00 -> 70.3 mm
- net Q4: track 0.00 -> 69.7 mm
- net Net-(R3-Pad1): track 0.00 -> 61.4 mm
- net CLOCK_OUT: track 0.00 -> 57.2 mm
- net Net-(C2-Pad1): track 0.00 -> 56.8 mm
- net Q2: track 0.00 -> 56.2 mm
- net Q1: track 0.00 -> 43.4 mm
- net Net-(SW1-Pad2): track 0.00 -> 28.7 mm
- net Net-(SW2-Pad2): track 0.00 -> 25.0 mm
- net Net-(R6-Pad2): track 0.00 -> 21.0 mm
- net Net-(C5-Pad1): track 0.00 -> 13.8 mm
- net Net-(R7-Pad1): track 0.00 -> 12.8 mm
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Other:
- board size 136.5 x 133.6 mm -> 102.8 x 128.4 mm

Commit message: update
Other:
- board text added: "1-0"
- board text added: "quiescent"
- board text added: "↑/↓"
- board text added: "►/►►"
Changed lines of the file:
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@@
       (outputformat 1)
       (mirror false)
-      (drillshape 1)
+      (drillshape 0)
       (scaleselection 1)
-      (outputdirectory "")
+      (outputdirectory "gerber/")
     )
   )
@@
     )
     (fp_line (start 3.95 -6.6) (end 3.95 6.6) (layer "F.Fab") (width 0.12))
+    (fp_line (start 3.95 -6.6) (end -3.95 -6.6) (layer "F.Fab") (width 0.12))
     (fp_line (start 3.95 6.6) (end -3.95 6.6) (layer "F.Fab") (width 0.12))
     (fp_line (start -3.95 -6.6) (end -3.95 6.6) (layer "F.Fab") (width 0.12))
-    (fp_line (start 3.95 -6.6) (end -3.95 -6.6) (layer "F.Fab") (width 0.12))
     (pad "" thru_hole circle locked (at 0 0 270) (size 7 7) (drill 6) (layers *.Cu *.Mask))
   )
@@
       (effects (font (size 1 1) (thickness 0.15)))
     )
-    (fp_line (start 3.95 -6.6) (end 3.95 6.6) (layer "F.Fab") (width 0.12))
-    (fp_line (start 3.95 6.6) (end -3.95 6.6) (layer "F.Fab") (width 0.12))
     (fp_line (start -3.95 -6.6) (end -3.95 6.6) (layer "F.Fab") (width 0.12))
     (fp_line (start 3.95 -6.6) (end -3.95 -6.6) (layer "F.Fab") (width 0.12))
+    (fp_line (start 3.95 6.6) (end -3.95 6.6) (layer "F.Fab") (width 0.12))
+    (fp_line (start 3.95 -6.6) (end 3.95 6.6) (layer "F.Fab") (width 0.12))
     (pad "" thru_hole circle locked (at 0 0 270) (size 7 7) (drill 6) (layers *.Cu *.Mask))
   )
@@
       (effects (font (size 1 1) (thickness 0.15)))
     )
+    (fp_line (start 5 12.98) (end 5 -1.42) (layer "F.CrtYd") (width 0.05))
     (fp_line (start 5 12.98) (end -5 12.98) (layer "F.CrtYd") (width 0.05))
     (fp_line (start 5 -1.42) (end -5 -1.42) (layer "F.CrtYd") (width 0.05))
     (fp_line (start -5 12.98) (end -5 -1.42) (layer "F.CrtYd") (width 0.05))
-    (fp_line (start 5 12.98) (end 5 -1.42) (layer "F.CrtYd") (width 0.05))
     (fp_line (start 0 0) (end 0 2.03) (layer "F.Fab") (width 0.1))
     (fp_line (start -4.5 12.48) (end -4.5 2.08) (layer "F.Fab") (width 0.1))
     (fp_line (start 4.5 2.03) (end -4.5 2.03) (layer "F.Fab") (width 0.1))
+    (fp_line (start 4.5 12.48) (end -4.5 12.48) (layer "F.Fab") (width 0.1))
     (fp_line (start 4.5 12.48) (end 4.5 2.08) (layer "F.Fab") (width 0.1))
-    (fp_line (start 4.5 12.48) (end -4.5 12.48) (layer "F.Fab") (width 0.1))
     (fp_circle (center 0 6.5) (end 4 6.5) (layer "F.Fab") (width 0.12) (fill none))
     (pad "" thru_hole circle locked (at 0 6.5 180) (size 7 7) (drill 6) (layers *.Cu *.Mask))
@@
       (effects (font (size 1 1) (thickness 0.15)))
     )
-    (fp_line (start 5 12.98) (end -5 12.98) (layer "F.CrtYd") (width 0.05))
-    (fp_line (start 5 -1.42) (end -5 -1.42) (layer "F.CrtYd") (width 0.05))
     (fp_line (start -5 12.98) (end -5 -1.42) (layer "F.CrtYd") (width 0.05))
     (fp_line (start 5 12.98) (end 5 -1.42) (layer "F.CrtYd") (width 0.05))
-    (fp_line (start 0 0) (end 0 2.03) (layer "F.Fab") (width 0.1))
+    (fp_line (start 5 -1.42) (end -5 -1.42) (layer "F.CrtYd") (width 0.05))
+    (fp_line (start 5 12.98) (end -5 12.98) (layer "F.CrtYd") (width 0.05))
     (fp_line (start -4.5 12.48) (end -4.5 2.08) (layer "F.Fab") (width 0.1))
+    (fp_line (start 4.5 12.48) (end -4.5 12.48) (layer "F.Fab") (width 0.1))
     (fp_line (start 4.5 2.03) (end -4.5 2.03) (layer "F.Fab") (width 0.1))
     (fp_line (start 4.5 12.48) (end 4.5 2.08) (layer "F.Fab") (width 0.1))
-    (fp_line (start 4.5 12.48) (end -4.5 12.48) (layer "F.Fab") (width 0.1))
+    (fp_line (start 0 0) (end 0 2.03) (layer "F.Fab") (width 0.1))
     (fp_circle (center 0 6.5) (end 4 6.5) (layer "F.Fab") (width 0.12) (fill none))
     (pad "" thru_hole circle locked (at 0 6.5 180) (size 7 7) (drill 6) (layers *.Cu *.Mask))
@@
       (effects (font (size 1 1) (thickness 0.15)))
     )
+    (fp_line (start -5 12.98) (end -5 -1.42) (layer "F.CrtYd") (width 0.05))
+    (fp_line (start 5 -1.42) (end -5 -1.42) (layer "F.CrtYd") (width 0.05))
     (fp_line (start 5 12.98) (end -5 12.98) (layer "F.CrtYd") (width 0.05))
-    (fp_line (start 5 -1.42) (end -5 -1.42) (layer "F.CrtYd") (width 0.05))
-    (fp_line (start -5 12.98) (end -5 -1.42) (layer "F.CrtYd") (width 0.05))
     (fp_line (start 5 12.98) (end 5 -1.42) (layer "F.CrtYd") (width 0.05))
-    (fp_line (start 0 0) (end 0 2.03) (layer "F.Fab") (width 0.1))
     (fp_line (start -4.5 12.48) (end -4.5 2.08) (layer "F.Fab") (width 0.1))
-    (fp_line (start 4.5 2.03) (end -4.5 2.03) (layer "F.Fab") (width 0.1))
     (fp_line (start 4.5 12.48) (end 4.5 2.08) (layer "F.Fab") (width 0.1))
     (fp_line (start 4.5 12.48) (end -4.5 12.48) (layer "F.Fab") (width 0.1))
+    (fp_line (start 0 0) (end 0 2.03) (layer "F.Fab") (width 0.1))
+    (fp_line (start 4.5 2.03) (end -4.5 2.03) (layer "F.Fab") (width 0.1))
     (fp_circle (center 0 6.5) (end 4 6.5) (layer "F.Fab") (width 0.12) (fill none))
     (pad "" thru_hole circle locked (at 0 6.5 180) (size 7 7) (drill 6) (layers *.Cu *.Mask))
@@
     )
     (fp_line (start 5 12.98) (end -5 12.98) (layer "F.CrtYd") (width 0.05))
+    (fp_line (start 5 12.98) (end 5 -1.42) (layer "F.CrtYd") (width 0.05))
     (fp_line (start 5 -1.42) (end -5 -1.42) (layer "F.CrtYd") (width 0.05))
     (fp_line (start -5 12.98) (end -5 -1.42) (layer "F.CrtYd") (width 0.05))
-    (fp_line (start 5 12.98) (end 5 -1.42) (layer "F.CrtYd") (width 0.05))
+    (fp_line (start 4.5 12.48) (end 4.5 2.08) (layer "F.Fab") (width 0.1))
+    (fp_line (start 4.5 2.03) (end -4.5 2.03) (layer "F.Fab") (width 0.1))
     (fp_line (start 0 0) (end 0 2.03) (layer "F.Fab") (width 0.1))
     (fp_line (start -4.5 12.48) (end -4.5 2.08) (layer "F.Fab") (width 0.1))
-    (fp_line (start 4.5 2.03) (end -4.5 2.03) (layer "F.Fab") (width 0.1))
-    (fp_line (start 4.5 12.48) (end 4.5 2.08) (layer "F.Fab") (width 0.1))
     (fp_line (start 4.5 12.48) (end -4.5 12.48) (layer "F.Fab") (width 0.1))
     (fp_circle (center 0 6.5) (end 4 6.5) (layer "F.Fab") (width 0.12) (fill none))
@@
       (effects (font (size 1 1) (thickness 0.15)))
     )
-    (fp_line (start 5 12.98) (end -5 12.98) (layer "F.CrtYd") (width 0.05))
-    (fp_line (start 5 -1.42) (end -5 -1.42) (layer "F.CrtYd") (width 0.05))
     (fp_line (start -5 12.98) (end -5 -1.42) (layer "F.CrtYd") (width 0.05))
     (fp_line (start 5 12.98) (end 5 -1.42) (layer "F.CrtYd") (width 0.05))
+    (fp_line (start 5 -1.42) (end -5 -1.42) (layer "F.CrtYd") (width 0.05))
+    (fp_line (start 5 12.98) (end -5 12.98) (layer "F.CrtYd") (width 0.05))
+    (fp_line (start 4.5 2.03) (end -4.5 2.03) (layer "F.Fab") (width 0.1))
     (fp_line (start 0 0) (end 0 2.03) (layer "F.Fab") (width 0.1))
     (fp_line (start -4.5 12.48) (end -4.5 2.08) (layer "F.Fab") (width 0.1))
-    (fp_line (start 4.5 2.03) (end -4.5 2.03) (layer "F.Fab") (width 0.1))
     (fp_line (start 4.5 12.48) (end 4.5 2.08) (layer "F.Fab") (width 0.1))
     (fp_line (start 4.5 12.48) (end -4.5 12.48) (layer "F.Fab") (width 0.1))
@@
     (fp_line (start -3.18 3.03) (end -1.98 3.03) (layer "F.Fab") (width 0.1))
     (fp_line (start -3.18 -4.1) (end -2.18 -5.1) (layer "F.Fab") (width 0.1))
-    (pad "1" thru_hole roundrect locked (at 0 0) (size 1.7 1.7) (drill 1) (layers *.Cu *.Mask) (roundrect_rratio 0.147059)
+    (pad "1" thru_hole roundrect locked (at 0 0) (size 1.7 1.7) (drill 1) (layers *.Cu *.Mask) (roundrect_rratio 0.1470588235)
       (net 7 "Net-(D1-Pad2)") (pinfunction "Pin_1") (pintype "passive"))
     (pad "2" thru_hole circle locked (at 2.54 0) (size 1.7 1.7) (drill 1) (layers *.Cu *.Mask)
@@
   (gr_circle (center 103.676136 114.046) (end 104.565136 115.824) (layer "Edge.Cuts") (width 0.1) (fill none))
   (gr_circle (center 75.355136 114.173) (end 76.244136 115.951) (layer "Edge.Cuts") (width 0.1) (fill none))
+  (gr_text "quiescent" (at 102.108 144.653) (layer "F.Cu")
+    (effects (font (size 1.5 1.5) (thickness 0.3)))
+  )
+  (gr_text "1-0" (at 103.759 64.643) (layer "F.SilkS")
+    (effects (font (size 3 3) (thickness 0.15)))
+  )
+  (gr_text "↑/↓" (at 75.057 64.643) (layer "F.SilkS")
+    (effects (font (size 4 4) (thickness 0.15)))
+  )
+  (gr_text "►/►►" (at 90.043 64.643) (layer "F.SilkS")
+    (effects (font (size 2 2) (thickness 0.15)))
+  )
   (segment locked (start 151.232 88.345) (end 151.232 89.5703) (width 0.25) (layer "F.Cu") (net 1))
   (segment locked (start 136.754 91.0837) (end 138.029 92.3587) (width 0.25) (layer "F.Cu") (net 1))
