File: AS3363/ASVCA/ASVCA.kicad_pcb (KiCad board)
At the start: 2 copper layers, 137.5 x 128.7 mm, 72 parts, among them J1 Conn_02x05_Counter_Clockwise, J10 CVIN1, J11 OUTPUT1, J12 Conn_01x14_Female, J13 Conn_01x14_Male, J2 INPUT3a, J3 INPUT3b, J4 CVIN3, J5 OUTPUT3, J6 INPUT2, J7 CVIN2, J8 OUTPUT2, J9 INPUT1, U1 AS3363, U2 TL074, U3 TL074, U4 TL074

Commit message: update
Other:
- board text added: "+"
- board text added: "quiescent"
- board text added: "↑"
- board text added: "→"
- board text added: "↓"
